Commit message: Getting rid of more warnings.

File: models/components.urdf.xacro (robot description, xacro)
@@ -224,5 +224,5 @@
       <origin xyz="-0.045 -0.3 0" rpy="${PI/2} 0 0"/>
       <axis xyz="0 0 1"/>
-      <limit effort="10" lower="-4.55" upper="1.25" velocity="2.0"/>
+      <limit effort="10" lower="-4.55" upper="1.8" velocity="2.0"/>
       <dynamics damping="${0.5*b}" friction="0"/>
     </joint>

File: robots/wam4.urdf.xacro (robot description, xacro)
@@ -1,4 +1,4 @@
 <robot name="wam"
-  xmlns:xacro="http://www.ros.org/wiki/xacro">
+  xmlns:xacro="http://ros.org/wiki/xacro">
   <!-- Includea all the WAM stuff -->
   <xacro:include filename="$(find barrett_model)/models/wam_top.urdf.xacro"/>

File: robots/wam4_stump.urdf.xacro (robot description, xacro)
@@ -1,4 +1,4 @@
 <robot name="wam"
-  xmlns:xacro="http://www.ros.org/wiki/xacro">
+  xmlns:xacro="http://ros.org/wiki/xacro">
   <!-- Includea all the WAM stuff -->
   <xacro:include filename="$(find barrett_model)/models/wam_top.urdf.xacro"/>

File: robots/wam7.urdf.xacro (robot description, xacro)
@@ -1,4 +1,4 @@
 <robot name="wam"
-  xmlns:xacro="http://www.ros.org/wiki/xacro">
+  xmlns:xacro="http://ros.org/wiki/xacro">
   <!-- Includea all the WAM stuff -->
   <xacro:include filename="$(find barrett_model)/models/wam_top.urdf.xacro"/>

File: robots/wam_4dof_wam_bhand.urdf.xacro (robot description, xacro)
@@ -1,6 +1,6 @@
 <robot name="wam"
-  xmlns:xacro="http://www.ros.org/wiki/xacro">
+  xmlns:xacro="http://ros.org/wiki/xacro">
   <!-- Includea all the WAM stuff -->
-  <include filename="$(find barrett_model)/models/wam_top.urdf.xacro"/>
+  <xacro:include filename="$(find barrett_model)/models/wam_top.urdf.xacro"/>
   <!-- Root link is in the world frame-->
   <link name = "world"/>

File: robots/wam_7dof_wam_bhand.urdf.xacro (robot description, xacro)
@@ -1,9 +1,9 @@
 <robot name="wam"
-  xmlns:xacro="http://www.ros.org/wiki/xacro">
+  xmlns:xacro="http://ros.org/wiki/xacro">
   <!-- Includea all the WAM stuff -->
-  <include filename="$(find barrett_model)/models/wam_top.urdf.xacro"/>
+  <xacro:include filename="$(find barrett_model)/models/wam_top.urdf.xacro"/>
   <!-- Root link is in the world frame-->
   <link name = "world"/>
-  <xacro:wam_7dof prefix="wam" parent_link="world" xyz="0.02 0.46 1" rpy="0 0 0" />
+  <xacro:wam_7dof prefix="wam" parent_link="world" xyz="0 0 0" rpy="0 0 0" />
   <xacro:bhand prefix="wam/bhand" parent_link="wam/wrist_palm_link" xyz="0 0 0.06" rpy="0 0 ${PI}"/>
 </robot>

Commit message: Updated joint limits to more closely match the OpenRAVE ones.

File: models/components.urdf.xacro (robot description, xacro)
@@ -100,5 +100,5 @@
       <origin xyz="0 0 0" rpy="${-PI/2} 0 0"/>
       <axis xyz="0 0 1"/>
-      <limit effort="60" lower="-1.985" upper="1.985" velocity="2.0"/>
+      <limit effort="60" lower="-1.972" upper="1.972" velocity="2.0"/>
       <dynamics damping="${0.5*b}" friction="0"/>
     </joint>
@@ -136,5 +136,5 @@
       <origin xyz="0 0 0" rpy="${PI/2} 0 0"/>
       <axis xyz="0 0 1"/>
-      <limit effort="45" lower="-2.8" upper="2.8" velocity="2.0"/>
+      <limit effort="45" lower="-2.74" upper="2.74" velocity="2.0"/>
       <dynamics damping="${1.5*b}" friction="0"/>
     </joint>
@@ -173,5 +173,5 @@
       <origin xyz="0.045 0 0.55" rpy="${-PI/2} 0 0"/>
       <axis xyz="0 0 1"/>
-      <limit effort="30" lower="-0.9" upper="${PI}" velocity="2.00"/>
+      <limit effort="30" lower="-0.87" upper="${PI}" velocity="2.00"/>
       <dynamics damping="${0.8*b}" friction="0"/>
     </joint>
@@ -224,5 +224,5 @@
       <origin xyz="-0.045 -0.3 0" rpy="${PI/2} 0 0"/>
       <axis xyz="0 0 1"/>
-      <limit effort="10" lower="-4.55" upper="1.8" velocity="2.0"/>
+      <limit effort="10" lower="-4.55" upper="1.3089" velocity="2.0"/>
       <dynamics damping="${0.5*b}" friction="0"/>
     </joint>
